File: PCB/PI_actuatorcontroller.kicad_pcb (KiCad board)
At the start: 2 copper layers, 106 x 60 mm, 42 parts, among them IC1 TLV9032QDGKRQ1, J1 ACTUATOR1, J3 Barrel_Jack_Switch, U1 INA381A1IDSGR

Commit message: pcb de terça-feira
Parts:
- added GNDPAD: TestPoint_Pad_D1.5mm, TestPoint:TestPoint_Pad_D1.5mm, F.Cu at (121.7, 91.6)
- CPS12_2, D3: moved to B.Cu
- moved D3 18.9 mm to (180.5, 104.4), turned to 90 degrees
- moved REF** 12.0 mm to (187.2, 116.0)
- moved REF** 12.0 mm to (187.2, 66.0)
- moved CPS12_1 8.81 mm to (174.5, 104.8)
- moved J3 8.71 mm to (191.5, 103.2)
- moved D2 6.84 mm to (182.9, 77.1)
- moved TPAR1 2.61 mm to (118.2, 90.6)
- moved CPS12_2 0.50 mm to (171.9, 105.0)
- moved RENA1 0.50 mm to (163.0, 75.5)
- moved REF** 0.06 mm to (104.2, 115.9)
Connections:
- CPS12_1 pad 1: Net-(D3-A) -> +12V
- CPS12_2 pad 1: Net-(D3-A) -> +12V
Routing:
- net Net-(D3-A): track 33.4 -> 7.19 mm
- net +12V: track 53.8 -> 69.3 mm, vias 0 -> 2
- net GND: track 295.4 -> 309.0 mm
- net Net-(D1-K): track 19.1 -> 9.99 mm
- net Net-(CR2-VBOOT): track 39.0 -> 42.2 mm
- net +3V3: track 62.2 -> 61.2 mm, vias 0 -> 1
- net /GPIO_RESET: track 7.77 -> 8.73 mm
- net Net-(CR2-OUT1A): track 16.7 -> 15.9 mm, vias 0 -> 1
- net /EnA_buf: track 44.0 -> 43.6 mm, vias 0 -> 2
- net Net-(CR2-OUT2A): vias 0 -> 1
Other:
- board size 106 x 60 mm -> 95.7 x 60 mm
