File: PCB/PI_actuatorcontroller.kicad_sch (KiCad schematic)
At the start: 38 parts, among them IC1 TLV9032QDGKRQ1, J1 ACTUATOR1, J3 Barrel_Jack_Switch, U1 INA381A1IDSGR

Commit message: pcb de terça-feira
Connections:
- net +12V: now also CPS12_1.1, CPS12_2.1
- net at D3.2 (A), J3.1: no longer CPS12_1.1, CPS12_2.1
Other:
- moved on the sheet: D3
Changed lines of the file:
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@@
+	)
+	(junction
+		(at 62.23 95.25)
+		(diameter 0)
+		(color 0 0 0 0)
+	)
+	(junction
+		(at 215.9 96.52)
+		(diameter 0)
+		(color 0 0 0 0)
+	)
+	(junction
+		(at 68.58 66.04)
+		(diameter 0)
+		(color 0 0 0 0)
+	)
+	(junction
+		(at 148.59 96.52)
+		(diameter 0)
+		(color 0 0 0 0)
+	)
+	(junction
+		(at 58.42 102.87)
+		(diameter 0)
+		(color 0 0 0 0)
 	)
 	(junction
@@
 	)
 	(junction
-		(at 62.23 95.25)
-		(diameter 0)
-		(color 0 0 0 0)
-	)
-	(junction
-		(at 215.9 96.52)
-		(diameter 0)
-		(color 0 0 0 0)
-	)
-	(junction
-		(at 68.58 66.04)
-		(diameter 0)
-		(color 0 0 0 0)
-	)
-	(junction
-		(at 148.59 96.52)
-		(diameter 0)
-		(color 0 0 0 0)
-	)
-	(junction
-		(at 58.42 102.87)
-		(diameter 0)
-		(color 0 0 0 0)
-	)
-	(junction
 		(at 105.41 44.45)
 		(diameter 0)
@@
 	(wire
 		(pts
-			(xy 35.56 95.25) (xy 54.61 95.25)
-		)
-		(stroke
-			(width 0)
-			(type default)
-		)
-	)
-	(wire
-		(pts
 			(xy 68.58 66.04) (xy 68.58 76.2)
 		)
@@
 	(wire
 		(pts
-			(xy 83.82 95.25) (xy 90.17 95.25)
-		)
-		(stroke
-			(width 0)
-			(type default)
-		)
-	)
-	(wire
-		(pts
 			(xy 58.42 102.87) (xy 62.23 102.87)
 		)
@@
 	(wire
 		(pts
+			(xy 54.61 95.25) (xy 62.23 95.25)
+		)
+		(stroke
+			(width 0)
+			(type default)
+		)
+	)
+	(wire
+		(pts
 			(xy 148.59 95.25) (xy 148.59 96.52)
 		)
@@
 	(wire
 		(pts
-			(xy 54.61 95.25) (xy 62.23 95.25)
-		)
-		(stroke
-			(width 0)
-			(type default)
-		)
-	)
-	(wire
-		(pts
 			(xy 105.41 44.45) (xy 109.22 44.45)
 		)
@@
 	(wire
 		(pts
+			(xy 35.56 95.25) (xy 38.1 95.25)
+		)
+		(stroke
+			(width 0)
+			(type default)
+		)
+	)
+	(wire
+		(pts
 			(xy 219.71 87.63) (xy 223.52 87.63)
 		)
@@
 	(wire
 		(pts
-			(xy 62.23 95.25) (xy 68.58 95.25)
+			(xy 62.23 95.25) (xy 90.17 95.25)
 		)
 		(stroke
@@
 		(pts
 			(xy 137.16 90.17) (xy 137.16 102.87)
+		)
+		(stroke
+			(width 0)
+			(type default)
+		)
+	)
+	(wire
+		(pts
+			(xy 53.34 95.25) (xy 54.61 95.25)
 		)
 		(stroke
@@
 	(symbol
 		(lib_id "STPST5H100AF:STPST5H100AF")
-		(at 86.36 95.25 180)
+		(at 55.88 95.25 180)
 		(unit 1)
 		(exclude_from_sim no)
@@
 		(fields_autoplaced yes)
 		(property "Reference" "D3"
-			(at 76.2 87.63 0)
+			(at 45.72 87.63 0)
 			(effects
 				(font
@@
 		)
 		(property "Value" "STPST5H100AF"
-			(at 76.2 90.17 0)
+			(at 45.72 90.17 0)
 			(effects
 				(font
@@
 		)
 		(property "Footprint" "STPST5H100AF:SODFL4724X103N"
-			(at 73.66 1.6 0)
+			(at 43.18 1.6 0)
 			(effects
 				(font
@@
 		)
 		(property "Datasheet" "https://www.st.com/resource/en/datasheet/stpst5h100.pdf"
-			(at 73.66 -98.4 0)
+			(at 43.18 -98.4 0)
 			(effects
 				(font
@@
 		)
 		(property "Description" "100 V, 5 A Power Schottky Trench Rectifier"
-			(at 86.36 95.25 0)
+			(at 55.88 95.25 0)
 			(effects
 				(font
@@
 		)
 		(property "Height" "1.03"
-			(at 73.66 -298.4 0)
+			(at 43.18 -298.4 0)
 			(effects
 				(font
@@
 		)
 		(property "Manufacturer_Name" "STMicroelectronics"
-			(at 73.66 -398.4 0)
+			(at 43.18 -398.4 0)
 			(effects
 				(font
@@
 		)
 		(property "Manufacturer_Part_Number" "STPST5H100AF"
-			(at 73.66 -498.4 0)
+			(at 43.18 -498.4 0)
 			(effects
 				(font
@@
 		)
 		(property "Arrow Part Number" ""
-			(at 73.66 -598.4 0)
+			(at 43.18 -598.4 0)
 			(effects
 				(font
@@
 		)
 		(property "Arrow Price/Stock" ""
-			(at 73.66 -698.4 0)
-			(effects
-				(font
+			(at 43.18 -698.4 0)
+			(effects
+				(font
