File: PCBcontrolador/PI_actuatorcontroller.kicad_sch (KiCad schematic)
At the start: 38 parts, among them IC1 TLV9032QDGKRQ1, J1 ACTUATOR1, J3 Barrel_Jack_Switch, U1 INA381A1IDSGR

Commit message: PCB controller final version
Parts:
- removed IC1: TLV9032QDGKRQ1, SOP65P490X110-8N, symbol TLV9032QDGKRQ1:TLV9032QDGKRQ1
- removed R4: 2k, Resistor_THT:R_Axial_DIN0207_L6.3mm_D2.5mm_P7.62mm_Horizontal, symbol Device:R
- removed TP3V3, TPAA1, TPCI2M1, TPCI2P1, TPCO2: TestPoint, TestPoint:TestPoint_Pad_D2.0mm, symbol Connector:TestPoint
- added TP1, TP2, TP3, TP3V3A1: TestPoint, TestPoint_THTPad_2.0x2.0mm_Drill1.0mm, symbol Connector:TestPoint
- R1, R3: value 2k -> 10K
- R2: value 2k -> 10k
- TPAAO1, TPAR1, TPHE1, TPHI1A1, TPHI1B1, TPHI2A1, TPHI2B1, TPHO1B1, TPHO2B1: footprint TestPoint:TestPoint_Pad_D2.0mm -> TestPoint_THTPad_2.0x2.0mm_Drill1.0mm
Connections:
- net EnA_buf is gone; now on net GPIO enable: RENA1.2
- net +3V3: now also R3.1, TP1.1; no longer RV1.1
- net GND: now also R1.2; no longer R3.1, RV1.3
- net GPIO enable: now also R2.1, U1.3 (*ALERT); no longer R2.2
- net at CR2.4 (OUT1A), J1.1: now also TP3.1
- net at CR2.18 (OUT2A), J1.2: now also TP2.1
- net at R3.2: now also RV1.1
- net at Cp1.1: now also CR2.19 (VCP); no longer Rp1.1
- net at CR2.12 (VBOOT), Cboot1.2: now also D2.1 (K); no longer D2.2 (A)
- net at Rp1.2: now also Cp1.2; no longer CR2.19 (VCP)
- net EnA_soft: no longer names the net of R1.1
- net EnA_soft: now also RV1.3
- removed net calert: R1.2, R2.1, U1.3 (*ALERT)
- new net: D1.1 (K), D2.2 (A), Rp1.1
- new net: R2.2, TP3V3A1.1
Other:
- moved on the sheet: Cp1, D2, R2, Rp1, TPHE1
