File: PCBsensor/PCBsensor.kicad_pcb (KiCad board)
At the start: 2 copper layers, 54.5 x 57.5 mm, 2 parts, among them U1 FMAMSDXX025WCSC3

Commit message: PCB sensor final version
Parts:
- added REF**: MountingHole_2.1mm, MountingHole:MountingHole_2.1mm, F.Cu at (152.9, 105.2)
- added REF**: MountingHole_2.1mm, MountingHole:MountingHole_2.1mm, F.Cu at (135.9, 105.2)
- added REF**: MountingHole_2.1mm, MountingHole:MountingHole_2.1mm, F.Cu at (152.9, 82.2)
- added REF**: MountingHole_2.1mm, MountingHole:MountingHole_2.1mm, F.Cu at (135.9, 82.2)
- added TP1: TestPoint, TestPoint:TestPoint_THTPad_2.0x2.0mm_Drill1.0mm, F.Cu at (136.5, 99.1)
- added TP2: TestPoint, TestPoint:TestPoint_THTPad_2.0x2.0mm_Drill1.0mm, F.Cu at (152.2, 99.1)
- added TP3: TestPoint, TestPoint:TestPoint_THTPad_2.0x2.0mm_Drill1.0mm, F.Cu at (143.9, 99.1)
- added TP4: TestPoint, TestPoint:TestPoint_THTPad_2.0x2.0mm_Drill1.0mm, F.Cu at (140.1, 99.1)
- added TP5: TestPoint, TestPoint:TestPoint_THTPad_2.0x2.0mm_Drill1.0mm, F.Cu at (148.4, 99.1)
Connections:
- U1 pad 1: unconnected-(U1-VP-Pad1) -> Net-(U1-VP)
- U1 pad 2: unconnected-(U1-SS-Pad2) -> Net-(U1-SS)
- U1 pad 3: GND -> Net-(U1-GND)
- U1 pad 4: unconnected-(U1-SCLK-Pad4) -> Net-(U1-SCLK)
- U1 pad 5: unconnected-(U1-MISO-Pad5) -> Net-(U1-MISO)
Routing:
- net unconnected-(U1-VP-Pad1): track 30.5 -> 0.00 mm
- net unconnected-(U1-MISO-Pad5): track 28.4 -> 0.00 mm
- net GND: track 23.6 -> 0.00 mm
- net unconnected-(U1-SCLK-Pad4): track 23.6 -> 0.00 mm
- net Net-(U1-VP): track 0.00 -> 18.9 mm
- net Net-(U1-SS): track 0.00 -> 18.9 mm
- net Net-(U1-MISO): track 0.00 -> 14.1 mm
- net Net-(U1-SCLK): track 0.00 -> 13.5 mm
- net Net-(U1-GND): track 0.00 -> 11.5 mm
Other:
- board size 54.5 x 57.5 mm -> 23 x 30 mm
