File: PCBsensor/PCBsensor.kicad_sch (KiCad schematic)
At the start: 1 part, among them U1 FMAMSDXX025WCSC3

Commit message: PCB sensor final version
Parts:
- added TP1, TP2, TP3, TP4, TP5: TestPoint, TestPoint:TestPoint_THTPad_2.0x2.0mm_Drill1.0mm, symbol Connector:TestPoint
Connections:
- net at U1.1 (VP): now also TP1.1
- net at U1.2 (SS): now also TP2.1
- net at U1.4 (SCLK): now also TP4.1
- net at U1.5 (MISO): now also TP5.1
- net GND: no longer names the net of U1.3 (GND)
- net GND: now also TP3.1
